Commit message: v1

File: src/circ_rover_description/urdf/rover_simple_v1_2.urdf (robot description, URDF)
Before this commit: robot rover_simple_v1_2, 21 links, 20 joints
Links:
- removed link BL_link
- removed link BR_link
- removed link FL_link
- removed link FR_link
- removed link L4low_link
- removed link L4up_link
- removed link LL2F_link
- removed link LL2M_link
- removed link LL2up_link
- removed link LL5Fup_link
- removed link LL5Mup_link
- removed link LL6up_link
- removed link ML_link
- removed link MR_link
- removed link RL2F_link
- removed link RL2M_link
- removed link RL2up_link
- removed link RL5Fup_link
- removed link RL5Mup_link
- removed link RL6up_link
- removed link base_link
- added link imu_link
- added link lidar_link; visual cylinder length=0.05 radius=0.05
Joints:
- removed joint BL_joint
- removed joint BR_joint
- removed joint FL_joint
- removed joint FR_joint
- removed joint L4low_joint
- removed joint L4up_joint
- removed joint LL2F_joint
- removed joint LL2M_joint
- removed joint LL2up_joint
- removed joint LL5Fup_joint
- removed joint LL5Mup_joint
- removed joint LL6up_joint
- removed joint ML_joint
- removed joint MR_joint
- removed joint RL2F_joint
- removed joint RL2M_joint
- removed joint RL2up_joint
- removed joint RL5Fup_joint
- removed joint RL5Mup_joint
- removed joint RL6up_joint
- added joint imu_joint: type fixed, parent base_link, child imu_link, origin xyz=0 0 0 rpy=0 0 0
- added joint lidar_joint: type fixed, parent base_link, child lidar_link, origin xyz=0.0 0.0 0.2 rpy=0 0 0
