Commit message: V1

File: src/circ_rover_description/urdf/rover.xacro (robot description, xacro)
@@ -1,152 +1,1375 @@
-<?xml version="1.0"?>
-<robot name="circ_rover" xmlns:xacro="http://ros.org/wiki/xacro">
-  <xacro:arg name="lidar_visualize" default="true" />
-  <!-- Include the base SolidWorks URDF -->
-  <xacro:include filename="$(find circ_rover_description)/urdf/rover_simple_v1_2.urdf" />
-  <!-- ============================================== -->
-  <!-- Gazebo Simulation Plugins & Properties         -->
-  <!-- ============================================== -->
-  <!-- Add basic friction and materials for the wheels -->
-  <xacro:macro name="wheel_gazebo_props" params="link_name">
-    <gazebo reference="${link_name}">
-      <mu1>0.8</mu1>
-      <mu2>0.8</mu2>
-      <material>Gazebo/DarkGrey</material>
-    </gazebo>
-  </xacro:macro>
-  <xacro:wheel_gazebo_props link_name="FL_link" />
-  <xacro:wheel_gazebo_props link_name="FR_link" />
-  <xacro:wheel_gazebo_props link_name="ML_link" />
-  <xacro:wheel_gazebo_props link_name="MR_link" />
-  <xacro:wheel_gazebo_props link_name="BL_link" />
-  <xacro:wheel_gazebo_props link_name="BR_link" />
-  <!-- Base link material -->
-  <gazebo reference="base_link">
-    <material>Gazebo/Grey</material>
-  </gazebo>
-  <!-- ============================================== -->
-  <!-- LiDAR Sensor (GPU Ray)                         -->
-  <!-- ============================================== -->
-  <!-- Assuming the LiDAR is mounted near the center top. We create a virtual link for it if it doesn't exist -->
-  <link name="lidar_link">
-    <visual>
-      <geometry>
-        <cylinder radius="0.05" length="0.05"/>
-      </geometry>
-      <material name="black">
-        <color rgba="0.1 0.1 0.1 1.0"/>
-      </material>
-    </visual>
-  </link>
-  <joint name="lidar_joint" type="fixed">
-    <parent link="base_link"/>
-    <child link="lidar_link"/>
-    <origin xyz="0.0 0.0 0.2" rpy="0 0 0"/>
-  </joint>
-  <gazebo reference="lidar_link">
-    <sensor name="lidar" type="ray">
-      <pose>0 0 0 0 0 0</pose>
-      <always_on>true</always_on>
-      <visualize>${lidar_visualize}</visualize>
-      <update_rate>10</update_rate>
-      <ray>
-        <scan>
-          <horizontal>
-            <samples>360</samples>
-            <resolution>1.000000</resolution>
-            <min_angle>-3.14159</min_angle>
-            <max_angle>3.14159</max_angle>
-          </horizontal>
-        </scan>
-        <range>
-          <min>0.12</min>
-          <max>12.0</max>
-          <resolution>0.015</resolution>
-        </range>
-        <noise>
-          <type>gaussian</type>
-          <mean>0.0</mean>
-          <stddev>0.01</stddev>
-        </noise>
-      </ray>
-      <plugin name="scan" filename="libgazebo_ros_ray_sensor.so">
-        <ros>
-          <remapping>~/out:=scan</remapping>
-        </ros>
-        <output_type>sensor_msgs/LaserScan</output_type>
-        <frame_name>lidar_link</frame_name>
-      </plugin>
-    </sensor>
-  </gazebo>
-  <!-- ============================================== -->
-  <!-- IMU Sensor                                     -->
-  <!-- ============================================== -->
-  <link name="imu_link"/>
-  <joint name="imu_joint" type="fixed">
-    <parent link="base_link"/>
-    <child link="imu_link"/>
-    <origin xyz="0 0 0" rpy="0 0 0"/>
-  </joint>
-  <gazebo reference="imu_link">
-    <sensor name="imu_sensor" type="imu">
-      <always_on>true</always_on>
-      <update_rate>100</update_rate>
-      <plugin name="imu_plugin" filename="libgazebo_ros_imu_sensor.so">
-        <ros>
-          <remapping>~/out:=imu/data_raw</remapping>
-        </ros>
-        <initial_orientation_as_reference>false</initial_orientation_as_reference>
-      </plugin>
-    </sensor>
-  </gazebo>
-  <!-- ============================================== -->
-  <!-- Joint State Publisher Plugin (for wheels)      -->
-  <!-- ============================================== -->
+<?xml version="1.0" encoding="utf-8"?>
+<!-- This URDF was automatically created by SolidWorks to URDF Exporter! Originally created by Stephen Brawner (brawner@gmail.com)
+     Commit Version: 1.6.0-4-g7f85cfe  Build Version: 1.6.7995.38578
+     For more information, please see http://wiki.ros.org/sw_urdf_exporter -->
+<robot
+  name="rover_simple_v1_2">
+  <link
+    name="base_link">
+    <inertial>
+      <origin
+        xyz="0.065394 3.6917E-17 -0.0291"
+        rpy="0 0 0" />
+      <mass
+        value="15.823" />
+      <inertia
+        ixx="0.3231"
+        ixy="-1.631E-16"
+        ixz="0.036909"
+        iyy="0.83124"
+        iyz="1.728E-17"
+        izz="1.1312" />
+    </inertial>
+    <visual>
+      <origin
+        xyz="0 0 0"
+        rpy="0 0 0" />
+      <geometry>
+        <mesh
+          filename="package://circ_rover_description/meshes/base_link.STL" />
+      </geometry>
+      <material
+        name="">
+        <color
+          rgba="0.79216 0.81961 0.93333 1" />
+      </material>
+    </visual>
+    <collision>
+      <origin
+        xyz="0 0 0"
+        rpy="0 0 0" />
+      <geometry>
+        <mesh
+          filename="package://circ_rover_description/meshes/base_link.STL" />
+      </geometry>
+    </collision>
+  </link>
+  <link
+    name="RL2up_link">
+    <inertial>
+      <origin
+        xyz="0.00098326 -0.048163 0.06572"
+        rpy="0 0 0" />
+      <mass
+        value="0.35165" />
+      <inertia
+        ixx="0.00058844"
+        ixy="4.4854E-07"
+        ixz="8.4163E-05"
+        iyy="0.0067323"
+        iyz="2.998E-05"
+        izz="0.0062126" />
+    </inertial>
+    <visual>
+      <origin
+        xyz="0 0 0"
+        rpy="0 0 0" />
+      <geometry>
+        <mesh
+          filename="package://circ_rover_description/meshes/RL2up_link.STL" />
+      </geometry>
+      <material
+        name="">
+        <color
+          rgba="0.79216 0.81961 0.93333 1" />
+      </material>
+    </visual>
+    <collision>
+      <origin
+        xyz="0 0 0"
+        rpy="0 0 0" />
+      <geometry>
+        <mesh
+          filename="package://circ_rover_description/meshes/RL2up_link.STL" />
+      </geometry>
+    </collision>
+  </link>
+  <joint
+    name="RL2up_joint"
+    type="revolute">
+    <origin
+      xyz="0.20894 -0.20857 -0.0127"
+      rpy="0 0 0" />
+    <parent
+      link="base_link" />
+    <child
+      link="RL2up_link" />
+    <axis
+      xyz="0 1 0" />
+    <limit
+      lower="-1.5"
+      upper="1.5"
+      effort="0"
+      velocity="0" />
+    <dynamics
+      damping="0.1"
+      friction="0.05" />
+  </joint>
+  <link
+    name="RL5Fup_link">
+    <inertial>
+      <origin
+        xyz="0.0076906 0.012145 -0.14103"
+        rpy="0 0 0" />
+      <mass
+        value="0.29333" />
+      <inertia
+        ixx="0.0028904"
+        ixy="-1.2514E-06"
+        ixz="-0.00017855"
+        iyy="0.0029492"
+        iyz="-2.79E-05"
+        izz="0.00010048" />
+    </inertial>
+    <visual>
+      <origin
+        xyz="0 0 0"
+        rpy="0 0 0" />
+      <geometry>
+        <mesh
+          filename="package://circ_rover_description/meshes/RL5Fup_link.STL" />
+      </geometry>
+      <material
+        name="">
+        <color
+          rgba="0.79216 0.81961 0.93333 1" />
+      </material>
+    </visual>
+    <collision>
+      <origin
+        xyz="0 0 0"
+        rpy="0 0 0" />
+      <geometry>
+        <mesh
+          filename="package://circ_rover_description/meshes/RL5Fup_link.STL" />
+      </geometry>
+    </collision>
+  </link>
+  <joint
+    name="RL5Fup_joint"
+    type="revolute">
+    <origin
+      xyz="0.21835 -0.0858 0.12175"
+      rpy="0 0 0" />
+    <parent
+      link="RL2up_link" />
+    <child
+      link="RL5Fup_link" />
+    <axis
+      xyz="0 1 0" />
+    <limit
+      lower="-1.5"
+      upper="1.5"
+      effort="0"
+      velocity="0" />
+    <dynamics
+      damping="0.1"
+      friction="0.05" />
+  </joint>
+  <link
+    name="FR_link">
+    <inertial>
+      <origin
+        xyz="0.00015846 0.04999 0.00043787"
+        rpy="0 0 0" />
+      <mass
+        value="3.1305" />
+      <inertia
+        ixx="0.010449"
+        ixy="-2.4542E-06"
+        ixz="2.8348E-06"
+        iyy="0.015699"
+        iyz="-6.782E-06"
+        izz="0.010455" />
+    </inertial>
+    <visual>
+      <origin
+        xyz="0 0 0"
+        rpy="0 0 0" />
+      <geometry>
+        <mesh
+          filename="package://circ_rover_description/meshes/FR_link.STL" />
+      </geometry>
+      <material
+        name="">
+        <color
+          rgba="0.69412 0.098039 0.098039 1" />
+      </material>
+    </visual>
+    <collision>
+      <origin
+        xyz="0 0 0"
+        rpy="0 0 0" />
+      <geometry>
+        <mesh
+          filename="package://circ_rover_description/meshes/FR_link.STL" />
+      </geometry>
+    </collision>
+  </link>
+  <joint
+    name="FR_joint"
+    type="continuous">
+    <origin
+      xyz="-0.000176 -0.1 -0.31299"
+      rpy="0 0 0" />
+    <parent
+      link="RL5Fup_link" />
+    <child
+      link="FR_link" />
+    <axis
+      xyz="0 1 0" />
+    <limit
+      lower="0"
+      upper="0"
+      effort="0"
+      velocity="0" />
+    <dynamics
+      friction="0.1" />
+  </joint>
+  <link
+    name="RL5Mup_link">
+    <inertial>
+      <origin
+        xyz="-0.00769063863242325 0.0121452936339811 -0.14103025565529"
+        rpy="0 0 0" />
+      <mass
+        value="0.293330883283669" />
+      <inertia
+        ixx="0.00289043444987535"
+        ixy="1.25138283176357E-06"
+        ixz="0.000178547994079131"
+        iyy="0.00294920584403958"
+        iyz="-2.79002722011482E-05"
+        izz="0.000100480286474077" />
+    </inertial>
+    <visual>
+      <origin
+        xyz="0 0 0"
+        rpy="0 0 0" />
+      <geometry>
+        <mesh
+          filename="package://circ_rover_description/meshes/RL5Mup_link.STL" />
+      </geometry>
+      <material
+        name="">
+        <color
+          rgba="0.792156862745098 0.819607843137255 0.933333333333333 1" />
+      </material>
+    </visual>
+    <collision>
+      <origin
+        xyz="0 0 0"
+        rpy="0 0 0" />
+      <geometry>
+        <mesh
+          filename="package://circ_rover_description/meshes/RL5Mup_link.STL" />
+      </geometry>
+    </collision>
+  </link>
+  <joint
+    name="RL5Mup_joint"
+    type="revolute">
+    <origin
+      xyz="-0.21461 -0.0858 0.12822"
+      rpy="0 0 0" />
+    <parent
+      link="RL2up_link" />
+    <child
+      link="RL5Mup_link" />
+    <axis
+      xyz="0 1 0" />
+    <limit
+      lower="-1.5"
+      upper="1.5"
+      effort="0"
+      velocity="0" />
+    <dynamics
+      damping="0.1"
+      friction="0.05" />
+    <mimic
+      joint="RL2up_joint"
+      multiplier="1"
+      offset="0" />
+  </joint>
+  <link
+    name="MR_link">
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
Commit message: Version_Mundos_GPS

File: src/circ_rover_description/urdf/rover.xacro (robot description, xacro)
@@ -100,4 +100,25 @@
   </gazebo>
   <!-- ============================================== -->
+  <!-- GPS Sensor                                     -->
+  <!-- ============================================== -->
+  <link name="gps_link"/>
+  <joint name="gps_joint" type="fixed">
+    <parent link="base_link"/>
+    <child link="gps_link"/>
+    <origin xyz="0 0 0.1" rpy="0 0 0"/>
+  </joint>
+  <gazebo reference="gps_link">
+    <sensor name="gps_sensor" type="gps">
+      <always_on>true</always_on>
+      <update_rate>10.0</update_rate>
+      <plugin name="gps_plugin" filename="libgazebo_ros_gps_sensor.so">
+        <ros>
+          <remapping>~/out:=gps/fix</remapping>
+        </ros>
+        <frame_name>gps_link</frame_name>
+      </plugin>
+    </sensor>
+  </gazebo>
+  <!-- ============================================== -->
   <!-- Joint State Publisher Plugin (for wheels)      -->
   <!-- ============================================== -->

Commit message: Revert "docs(sim): document world selector; add self-contained worlds"
This reverts commit 2bd341318eea89e9371ab629619de5a33093234b, reversing
changes made to 88758ab141491d218259aa84fba6efc983567fa4.

File: src/circ_rover_description/urdf/rover.xacro (robot description, xacro)
@@ -1,32 +1,24 @@
-<?xml version="1.0"?>
-<robot name="circ_rover" xmlns:xacro="http://ros.org/wiki/xacro">
-  <!-- Include the base SolidWorks URDF -->
-  <xacro:include filename="$(find circ_rover_description)/urdf/rover_simple_v1_2.urdf" />
-  <!-- ============================================== -->
-  <!-- Gazebo Simulation Plugins & Properties         -->
-  <!-- ============================================== -->
-  <!-- Add basic friction and materials for the wheels -->
-  <xacro:macro name="wheel_gazebo_props" params="link_name">
-    <gazebo reference="${link_name}">
-      <mu1>0.8</mu1>
-      <mu2>0.8</mu2>
-      <material>Gazebo/DarkGrey</material>
-    </gazebo>
-  </xacro:macro>
-  <xacro:wheel_gazebo_props link_name="FL_link" />
-  <xacro:wheel_gazebo_props link_name="FR_link" />
-  <xacro:wheel_gazebo_props link_name="ML_link" />
-  <xacro:wheel_gazebo_props link_name="MR_link" />
-  <xacro:wheel_gazebo_props link_name="BL_link" />
-  <xacro:wheel_gazebo_props link_name="BR_link" />
-  <!-- Base link material -->
-  <gazebo reference="base_link">
-    <material>Gazebo/Grey</material>
-  </gazebo>
-  <!-- ============================================== -->
-  <!-- LiDAR Sensor (GPU Ray)                         -->
-  <!-- ============================================== -->
-  <!-- Assuming the LiDAR is mounted near the center top. We create a virtual link for it if it doesn't exist -->
-  <link name="lidar_link">
+<?xml version="1.0" encoding="utf-8"?>
+<!-- This URDF was automatically created by SolidWorks to URDF Exporter! Originally created by Stephen Brawner (brawner@gmail.com)
+     Commit Version: 1.6.0-4-g7f85cfe  Build Version: 1.6.7995.38578
+     For more information, please see http://wiki.ros.org/sw_urdf_exporter -->
+<robot
+  name="rover_simple_v1_2">
+  <link
+    name="base_link">
+    <inertial>
+      <origin
+        xyz="0.065394 3.6917E-17 -0.0291"
+        rpy="0 0 0" />
+      <mass
+        value="15.823" />
+      <inertia
+        ixx="0.3231"
+        ixy="-1.631E-16"
+        ixz="0.036909"
+        iyy="0.83124"
+        iyz="1.728E-17"
+        izz="1.1312" />
+    </inertial>
     <visual>
       <origin
@@ -114,84 +106,1136 @@
       friction="0.05" />
   </joint>
-  <gazebo reference="lidar_link">
-    <sensor name="lidar" type="ray">
-      <pose>0 0 0 0 0 0</pose>
-      <always_on>true</always_on>
-      <visualize>true</visualize>
-      <update_rate>10</update_rate>
-      <ray>
-        <scan>
-          <horizontal>
-            <samples>360</samples>
-            <resolution>1.000000</resolution>
-            <min_angle>-3.14159</min_angle>
-            <max_angle>3.14159</max_angle>
-          </horizontal>
-        </scan>
-        <range>
-          <min>0.12</min>
-          <max>12.0</max>
-          <resolution>0.015</resolution>
-        </range>
-        <noise>
-          <type>gaussian</type>
-          <mean>0.0</mean>
-          <stddev>0.01</stddev>
-        </noise>
-      </ray>
-      <plugin name="scan" filename="libgazebo_ros_ray_sensor.so">
-        <ros>
-          <remapping>~/out:=scan</remapping>
-        </ros>
-        <output_type>sensor_msgs/LaserScan</output_type>
-        <frame_name>lidar_link</frame_name>
-      </plugin>
-    </sensor>
-  </gazebo>
-  <!-- ============================================== -->
-  <!-- IMU Sensor                                     -->
-  <!-- ============================================== -->
-  <link name="imu_link"/>
-  <joint name="imu_joint" type="fixed">
-    <parent link="base_link"/>
-    <child link="imu_link"/>
-    <origin xyz="0 0 0" rpy="0 0 0"/>
-  </joint>
-  <gazebo reference="imu_link">
-    <sensor name="imu_sensor" type="imu">
-      <always_on>true</always_on>
-      <update_rate>100</update_rate>
-      <plugin name="imu_plugin" filename="libgazebo_ros_imu_sensor.so">
-        <ros>
-          <remapping>~/out:=imu/data_raw</remapping>
-        </ros>
-        <initial_orientation_as_reference>false</initial_orientation_as_reference>
-      </plugin>
-    </sensor>
-  </gazebo>
-  <!-- ============================================== -->
-  <!-- GPS Sensor                                     -->
-  <!-- ============================================== -->
-  <link name="gps_link"/>
-  <joint name="gps_joint" type="fixed">
-    <parent link="base_link"/>
-    <child link="gps_link"/>
-    <origin xyz="0 0 0.1" rpy="0 0 0"/>
-  </joint>
-  <gazebo reference="gps_link">
-    <sensor name="gps_sensor" type="gps">
-      <always_on>true</always_on>
-      <update_rate>10.0</update_rate>
-      <plugin name="gps_plugin" filename="libgazebo_ros_gps_sensor.so">
-        <ros>
-          <remapping>~/out:=gps/fix</remapping>
-        </ros>
-        <frame_name>gps_link</frame_name>
-      </plugin>
-    </sensor>
-  </gazebo>
-  <!-- ============================================== -->
-  <!-- Joint State Publisher Plugin (for wheels)      -->
-  <!-- ============================================== -->
+  <link
+    name="RL5Fup_link">
+    <inertial>
+      <origin
+        xyz="0.0076906 0.012145 -0.14103"
+        rpy="0 0 0" />
+      <mass
+        value="0.29333" />
+      <inertia
+        ixx="0.0028904"
+        ixy="-1.2514E-06"
+        ixz="-0.00017855"
+        iyy="0.0029492"
+        iyz="-2.79E-05"
+        izz="0.00010048" />
+    </inertial>
+    <visual>
+      <origin
+        xyz="0 0 0"
+        rpy="0 0 0" />
+      <geometry>
+        <mesh
+          filename="package://circ_rover_description/meshes/RL5Fup_link.STL" />
+      </geometry>
+      <material
+        name="">
+        <color
+          rgba="0.79216 0.81961 0.93333 1" />
+      </material>
+    </visual>
+    <collision>
+      <origin
+        xyz="0 0 0"
+        rpy="0 0 0" />
+      <geometry>
+        <mesh
+          filename="package://circ_rover_description/meshes/RL5Fup_link.STL" />
+      </geometry>
+    </collision>
+  </link>
+  <joint
+    name="RL5Fup_joint"
+    type="revolute">
+    <origin
+      xyz="0.21835 -0.0858 0.12175"
+      rpy="0 0 0" />
+    <parent
+      link="RL2up_link" />
+    <child
+      link="RL5Fup_link" />
+    <axis
+      xyz="0 1 0" />
+    <limit
+      lower="-1.5"
+      upper="1.5"
+      effort="0"
+      velocity="0" />
+    <dynamics
+      damping="0.1"
+      friction="0.05" />
+  </joint>
+  <link
+    name="FR_link">
+    <inertial>
+      <origin
+        xyz="0.00015846 0.04999 0.00043787"
+        rpy="0 0 0" />
+      <mass
+        value="3.1305" />
+      <inertia
+        ixx="0.010449"
+        ixy="-2.4542E-06"
+        ixz="2.8348E-06"
+        iyy="0.015699"
+        iyz="-6.782E-06"
+        izz="0.010455" />
+    </inertial>
+    <visual>
+      <origin
+        xyz="0 0 0"
+        rpy="0 0 0" />
+      <geometry>
+        <mesh
+          filename="package://circ_rover_description/meshes/FR_link.STL" />
+      </geometry>
+      <material
+        name="">
+        <color
+          rgba="0.69412 0.098039 0.098039 1" />
+      </material>
+    </visual>
+    <collision>
+      <origin
+        xyz="0 0 0"
+        rpy="0 0 0" />
+      <geometry>
+        <mesh
+          filename="package://circ_rover_description/meshes/FR_link.STL" />
+      </geometry>
+    </collision>
+  </link>
+  <joint
+    name="FR_joint"
+    type="continuous">
+    <origin
+      xyz="-0.000176 -0.1 -0.31299"
+      rpy="0 0 0" />
+    <parent
+      link="RL5Fup_link" />
+    <child
+      link="FR_link" />
+    <axis
+      xyz="0 1 0" />
+    <limit
+      lower="0"
+      upper="0"
+      effort="0"
+      velocity="0" />
+    <dynamics
+      friction="0.1" />
+  </joint>
+  <link
+    name="RL5Mup_link">
+    <inertial>
+      <origin
+        xyz="-0.00769063863242325 0.0121452936339811 -0.14103025565529"
+        rpy="0 0 0" />
+      <mass
+        value="0.293330883283669" />
+      <inertia
+        ixx="0.00289043444987535"
+        ixy="1.25138283176357E-06"
+        ixz="0.000178547994079131"
+        iyy="0.00294920584403958"
+        iyz="-2.79002722011482E-05"
+        izz="0.000100480286474077" />
+    </inertial>
+    <visual>
+      <origin
+        xyz="0 0 0"
+        rpy="0 0 0" />
+      <geometry>
+        <mesh
+          filename="package://circ_rover_description/meshes/RL5Mup_link.STL" />
+      </geometry>
+      <material
+        name="">
+        <color
+          rgba="0.792156862745098 0.819607843137255 0.933333333333333 1" />
+      </material>
+    </visual>
+    <collision>
+      <origin
+        xyz="0 0 0"
+        rpy="0 0 0" />
+      <geometry>
+        <mesh
+          filename="package://circ_rover_description/meshes/RL5Mup_link.STL" />
+      </geometry>
+    </collision>
+  </link>
+  <joint
+    name="RL5Mup_joint"
+    type="revolute">
+    <origin
+      xyz="-0.21461 -0.0858 0.12822"
+      rpy="0 0 0" />
+    <parent
+      link="RL2up_link" />
+    <child
+      link="RL5Mup_link" />
+    <axis
+      xyz="0 1 0" />
+    <limit
+      lower="-1.5"
+      upper="1.5"
+      effort="0"
+      velocity="0" />
+    <dynamics
+      damping="0.1"
+      friction="0.05" />
+    <mimic
+      joint="RL2up_joint"
+      multiplier="1"
+      offset="0" />
+  </joint>
+  <link
+    name="MR_link">
+    <inertial>
+      <origin
+        xyz="-4.4033E-05 0.04999 0.00046357"
+        rpy="0 0 0" />
+      <mass
+        value="3.1305" />
+      <inertia
+        ixx="0.010448"
+        ixy="6.82E-07"
+        ixz="-6.7415E-07"
+        iyy="0.015699"
+        iyz="-7.1801E-06"
+        izz="0.010456" />
+    </inertial>
+    <visual>
+      <origin
+        xyz="0 0 0"
+        rpy="0 0 0" />
+      <geometry>
+        <mesh
+          filename="package://circ_rover_description/meshes/MR_link.STL" />
+      </geometry>
+      <material
+        name="">
+        <color
+          rgba="0.69412 0.098039 0.098039 1" />
+      </material>
+    </visual>
+    <collision>
+      <origin
+        xyz="0 0 0"
+        rpy="0 0 0" />
+      <geometry>
+        <mesh
+          filename="package://circ_rover_description/meshes/MR_link.STL" />
+      </geometry>
+    </collision>
+  </link>
+  <joint
+    name="MR_joint"
+    type="continuous">
+    <origin
+      xyz="4.8996E-05 -0.1 -0.31301"
+      rpy="0 0 0" />
+    <parent
+      link="RL5Mup_link" />
+    <child
+      link="MR_link" />
+    <axis
+      xyz="0 1 0" />
+    <dynamics
+      friction="0.1" />
+  </joint>
+  <link
+    name="RL2F_link">
+    <inertial>
+      <origin
+        xyz="0.10918 -0.0477 0.060874"
+        rpy="0 0 0" />
+      <mass
+        value="0.18497" />
+      <inertia
+        ixx="0.00031847"
+        ixy="3.5529E-05"
+        ixz="-0.00051774"
+        iyy="0.0012362"
+        iyz="1.981E-05"
+        izz="0.00095834" />
+    </inertial>
+    <visual>
+      <origin
+        xyz="0 0 0"
+        rpy="0 0 0" />
+      <geometry>
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